File: pcb/open_game_pad_classic/open_game_pad_classic.kicad_pcb (KiCad board)
At the start: 2 copper layers, 0 parts

Commit message: Updated the PCB and scheme. 2-layered, ground plane.
Parts:
- added AMP1: LM358, LM358:DIL8, F.Cu at (145.1, 89.3)
- added C1: 100nF, Capacitor_SMD:C_0201_0603Metric, F.Cu at (143.0, 67.3)
- added C2: 0.01 mkF, Capacitor_SMD:C_0201_0603Metric, F.Cu at (124.7, 73.7)
- added C3: 0.1 mkF, Capacitor_SMD:C_0201_0603Metric, F.Cu at (122.8, 73.7)
- added CR1: 74HC163, Package_SO:SOIC-16W_7.5x10.3mm_P1.27mm, F.Cu at (157.6, 90.5)
- added D1: 3v6, Diode_SMD:D_MiniMELF, F.Cu at (156.8, 58.6)
- added D2: 3v6, Diode_SMD:D_MiniMELF, F.Cu at (154.0, 58.6)
- added J1: COM-09032, COM-09032:XDCR_COM-09032, F.Cu at (170.0, 110.0)
- added J2: COM-09032, COM-09032:XDCR_COM-09032, F.Cu at (120.0, 110.0)
- added R1: R 5.1K, Resistor_SMD:R_0402_1005Metric, F.Cu at (152.0, 61.5)
- added R10: R 10K, Resistor_SMD:R_0805_2012Metric, F.Cu at (138.4, 86.6)
- added R2: R 5.1K, Resistor_SMD:R_0402_1005Metric, F.Cu at (139.7, 62.0)
- added R3: R 75, Resistor_SMD:R_0402_1005Metric, F.Cu at (145.7, 67.0)
- added R4: R 75, Resistor_SMD:R_0402_1005Metric, F.Cu at (144.4, 66.0)
- added R5: R 1.5K, Resistor_SMD:R_0603_1608Metric, F.Cu at (144.4, 70.3)
- added R6: R 10K, Resistor_SMD:R_0402_1005Metric, F.Cu at (142.8, 68.7)
- added R7: R 10K, Resistor_SMD:R_0402_1005Metric, F.Cu at (145.3, 95.1)
- added R8: R 4.7K, Resistor_SMD:R_0402_1005Metric, F.Cu at (136.3, 91.8)
- added R9: R 4.7K, Resistor_SMD:R_0402_1005Metric, F.Cu at (136.3, 89.2)
- added REG1: 74HC165, Package_SO:SOIC-16_3.9x9.9mm_P1.27mm, F.Cu at (126.3, 90.4)
- added SW1: ~, TS02-66-95-BK-260-LCR-D:SW_TS02-66-95-BK-260-LCR-D, F.Cu at (125.0, 70.0)
- added SW10: ~, TS02-66-95-BK-260-LCR-D:SW_TS02-66-95-BK-260-LCR-D, F.Cu at (211.2, 84.0)
- added SW11: ~, TS02-66-95-BK-260-LCR-D:SW_TS02-66-95-BK-260-LCR-D, F.Cu at (201.0, 61.0)
- added SW12: ~, TS02-66-95-BK-260-LCR-D:SW_TS02-66-95-BK-260-LCR-D, F.Cu at (137.9, 80.0)
- added SW13: ~, TS02-66-95-BK-260-LCR-D:SW_TS02-66-95-BK-260-LCR-D, F.Cu at (196.2, 99.0)
- added SW14: ~, TS02-66-95-BK-260-LCR-D:SW_TS02-66-95-BK-260-LCR-D, F.Cu at (98.0, 94.0)
- added SW15: ~, TS02-66-95-BK-260-LCR-D:SW_TS02-66-95-BK-260-LCR-D, F.Cu at (165.0, 70.0)
- added SW16: ~, TS02-66-95-BK-260-LCR-D:SW_TS02-66-95-BK-260-LCR-D, F.Cu at (152.2, 80.0)
- added SW2: ~, TS02-66-95-BK-260-LCR-D:SW_TS02-66-95-BK-260-LCR-D, F.Cu at (93.0, 61.2)
- added SW3: ~, TS02-66-95-BK-260-LCR-D:SW_TS02-66-95-BK-260-LCR-D, F.Cu at (88.0, 84.0)
- added SW4: ~, TS02-66-95-BK-260-LCR-D:SW_TS02-66-95-BK-260-LCR-D, F.Cu at (181.2, 84.0)
- added SW5: ~, TS02-66-95-BK-260-LCR-D:SW_TS02-66-95-BK-260-LCR-D, F.Cu at (103.0, 61.2)
- added SW6: ~, TS02-66-95-BK-260-LCR-D:SW_TS02-66-95-BK-260-LCR-D, F.Cu at (98.0, 74.0)
- added SW7: ~, TS02-66-95-BK-260-LCR-D:SW_TS02-66-95-BK-260-LCR-D, F.Cu at (196.2, 69.0)
- added SW8: ~, TS02-66-95-BK-260-LCR-D:SW_TS02-66-95-BK-260-LCR-D, F.Cu at (191.0, 61.0)
- added SW9: ~, TS02-66-95-BK-260-LCR-D:SW_TS02-66-95-BK-260-LCR-D, F.Cu at (108.0, 84.0)
- added U1: MM74C923, Package_SO:SOIC-20W_7.5x12.8mm_P1.27mm, F.Cu at (125.0, 80.0)
- added U2: 74HC4051, Package_SO:TSSOP-16_4.4x5mm_P0.65mm, F.Cu at (145.2, 98.6)
- added U3: SN74AHC1G04DBVR, SN74AHC1G04DBVR:SOT95P280X145-5N, F.Cu at (131.7, 96.4)
- added USB1: USB_C_Receptacle_USB2.0_14P, Connector_USB:USB_C_Receptacle_HCTL_HC-TYPE-C-16P-01A, F.Cu at (145.7, 60.0)
- added mC1: ATtiny85V-20u, Package_SO:SOIC-8W_5.3x5.3mm_P1.27mm, F.Cu at (145.1, 78.8)
Routing:
- net /X2: track 0.00 -> 223.3 mm, vias 0 -> 4
- net /X1: track 0.00 -> 189.6 mm, vias 0 -> 2
- net +5V: track 0.00 -> 176.9 mm, vias 0 -> 2
- net /Y3: track 0.00 -> 167.6 mm, vias 0 -> 1
- net /X3: track 0.00 -> 161.4 mm, vias 0 -> 4
- net /Y4: track 0.00 -> 145.3 mm, vias 0 -> 4
- net /Y1: track 0.00 -> 141.3 mm, vias 0 -> 1
- net /Y2: track 0.00 -> 138.9 mm, vias 0 -> 3
- net /X4: track 0.00 -> 131.8 mm, vias 0 -> 3
- net /Y5: track 0.00 -> 100.9 mm, vias 0 -> 2
- net Net-(J1-V): track 0.00 -> 51.0 mm, vias 0 -> 2
- net Net-(REG1-~{PL}): track 0.00 -> 39.3 mm
- net Net-(J1-H): track 0.00 -> 37.8 mm, vias 0 -> 2
- net /DIN: track 0.00 -> 37.4 mm, vias 0 -> 2
- net /CLK: track 0.00 -> 30.2 mm
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- added copper zone on B.Cu, net GND
- added copper zone on F.Cu, net GND
Other:
- board outline added: 140 x 70 mm
