File: pcb/open_game_pad_classic/open_game_pad_classic.kicad_pcb (KiCad board)
At the start: 2 copper layers, 140 x 71 mm, 54 parts, among them J1 COM-09032, J2 COM-09032

Commit message: Added the logo.
Parts:
- added G***: LOGO, LOGO, F.Cu at (167.0, 88.0)
